File: klasesdarbs/ONE_TRAN_AMP.kicad_pcb (KiCad board)
At the start: 2 copper layers, 52.1 x 30.5 mm, 11 parts, among them J1 Signal in, J2 Signal out, J3 Power, Q1 BC547

Commit message: course work
Parts:
- added G***: LOGO, Battery_holders:BrEE_LOGO_0_5_inch, F.Cu at (130.8, 105.4)
- moved R3 16.3 mm to (148.6, 105.4), turned to 270 degrees
- moved R4 16.3 mm to (152.4, 105.4), turned to 270 degrees
- moved R1 11.4 mm to (148.6, 101.6)
- moved R2 11.4 mm to (152.4, 101.6)
- moved C2 10.2 mm to (137.2, 97.8)
- moved C3 9.06 mm to (138.4, 113.0)
- moved Q1 1.80 mm to (143.5, 105.4), turned to 0 degrees
- moved C1 1.27 mm to (125.8, 97.8)
- moved J2 0.11 mm to (162.6, 109.2)
- moved J3 0.08 mm to (162.6, 96.5)
Routing:
- net GND: track 78.7 -> 0.00 mm
- net Net-(J3-Pad2): track 45.2 -> 18.9 mm
- net Net-(C1-Pad1): track 27.2 -> 45.0 mm
- net Net-(C3-Pad2): track 11.3 -> 20.2 mm
- net Net-(C3-Pad1): track 13.4 -> 16.9 mm
- net Net-(C1-Pad2): track 12.6 -> 13.8 mm
Other:
- net class Power: trace_width 0.5 -> 0.3
