File: Clock_LCD/Clock_LCD.kicad_pcb (KiCad board)
At the start: 2 copper layers, 21 parts, among them J1 Conn_01x01, J2 Conn_01x01, SW1 Reset, U1 LM7805_TO220, U2 ATMEGA328P-PU, U3 DS1307+, Y1 16MHz, Y2 32,768KHz

Commit message: komponenetes vietas izmaina
Parts:
- moved BT1 35.6 mm to (177.6, 97.8)
Changed lines of the file:
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@@
     (links 51)
     (no_connects 51)
-    (area 0 0 0 0)
+    (area 66.372381 26.595 225.125074 163.35)
     (thickness 1.6)
     (drawings 0)
@@
   )
   (module Battery_Holders:Keystone_103_1x20mm-CoinCell (layer F.Cu)
-    (at 197.95 68.58)
+    (at 177.63 97.79)
     (descr http://www.keyelco.com/product-pdf.cfm?p=719)
     (tags "Keystone type 103 battery holder")
